Commit message: Slam and Mapping

File: vehicle_description/urdf/body.xacro (robot description, xacro)
@@ -4,6 +4,6 @@
   <xacro:include filename="$(find vehicle_description)/urdf/wheels.xacro"/>
   <xacro:include filename="$(find vehicle_description)/urdf/differential.xacro"/>
-  <xacro:property name="pi" value="3.1415926535897931"/>
   <xacro:include filename="$(find vehicle_description)/urdf/lidar.xacro"/>
+  <xacro:property name="pi" value="3.1415926535897931" scope="global"/>
   <!-- Base Link -->
   <xacro:base_link/>
@@ -18,4 +18,7 @@
   <!-- Control Systems -->
   <xacro:differential_drive/>
-  <xacro:lidar_sensor name="hokuyo" parent="base_link" xyz="0.3 0 0.2" rpy="0 0 0"/>
+  <!-- IMPORTANT: Add the transmissions -->
+  <xacro:wheel_transmissions/>
+  <!-- LiDAR Sensor -->
+  <xacro:lidar_sensor name="hokuyo" parent="base_link" xyz="0.3 0 0.4" rpy="0 0 0"/>
 </robot>

File: vehicle_description/urdf/differential.xacro (robot description, xacro)
@@ -6,4 +6,5 @@
       <plugin name="gazebo_ros_control" filename="libgazebo_ros_control.so">
         <robotNamespace>/</robotNamespace>
+        <robotSimType>gazebo_ros_control/DefaultRobotHWSim</robotSimType>
       </plugin>
     </gazebo>
@@ -24,29 +25,33 @@
         <publishWheelTF>false</publishWheelTF>
         <publishOdomTF>true</publishOdomTF>
+        <publishWheelJointState>true</publishWheelJointState>
+        <legacyMode>false</legacyMode>
       </plugin>
     </gazebo>
-    <!-- Transmission for ROS Control -->
-    <xacro:macro name="wheel_transmissions">
-      <transmission name="left_wheel_trans">
-        <type>transmission_interface/SimpleTransmission</type>
-        <joint name="left_wheel_joint">
-          <hardwareInterface>hardware_interface/VelocityJointInterface</hardwareInterface>
-        </joint>
-        <actuator name="left_wheel_motor">
-          <hardwareInterface>hardware_interface/VelocityJointInterface</hardwareInterface>
-          <mechanicalReduction>1</mechanicalReduction>
-        </actuator>
-      </transmission>
-      <transmission name="right_wheel_trans">
-        <type>transmission_interface/SimpleTransmission</type>
-        <joint name="right_wheel_joint">
-          <hardwareInterface>hardware_interface/VelocityJointInterface</hardwareInterface>
-        </joint>
-        <actuator name="right_wheel_motor">
-          <hardwareInterface>hardware_interface/VelocityJointInterface</hardwareInterface>
-          <mechanicalReduction>1</mechanicalReduction>
-        </actuator>
-      </transmission>
-    </xacro:macro>
+    <!-- Call the transmission macro -->
+    <xacro:wheel_transmissions/>
+  </xacro:macro>
+  <!-- Transmission for ROS Control -->
+  <xacro:macro name="wheel_transmissions">
+    <transmission name="left_wheel_trans">
+      <type>transmission_interface/SimpleTransmission</type>
+      <joint name="left_wheel_joint">
+        <hardwareInterface>hardware_interface/VelocityJointInterface</hardwareInterface>
+      </joint>
+      <actuator name="left_wheel_motor">
+        <hardwareInterface>hardware_interface/VelocityJointInterface</hardwareInterface>
+        <mechanicalReduction>1</mechanicalReduction>
+      </actuator>
+    </transmission>
+    <transmission name="right_wheel_trans">
+      <type>transmission_interface/SimpleTransmission</type>
+      <joint name="right_wheel_joint">
+        <hardwareInterface>hardware_interface/VelocityJointInterface</hardwareInterface>
+      </joint>
+      <actuator name="right_wheel_motor">
+        <hardwareInterface>hardware_interface/VelocityJointInterface</hardwareInterface>
+        <mechanicalReduction>1</mechanicalReduction>
+      </actuator>
+    </transmission>
   </xacro:macro>
 </robot>

File: vehicle_description/urdf/lidar.xacro (robot description, xacro)
@@ -1,6 +1,6 @@
 <?xml version="1.0"?>
 <robot xmlns:xacro="http://www.ros.org/wiki/xacro">
-<!-- This should be at the top of lidar.xacro -->
-<xacro:property name="pi" value="3.1415926535897931"/>
+<!-- In both body.xacro and lidar.xacro -->
+  <xacro:property name="pi" value="3.1415926535897931" scope="global"/>
   <xacro:macro name="lidar_sensor" params="name parent xyz rpy">
     <link name="${name}_link">
@@ -34,5 +34,5 @@
         <pose>0 0 0 0 0 0</pose>
         <visualize>true</visualize>
-        <update_rate>40</update_rate>
+        <update_rate>12</update_rate>
         <ray>
           <scan>
@@ -46,5 +46,5 @@
           <range>
             <min>0.10</min>
-            <max>30.0</max>
+            <max>12.0</max>
             <resolution>0.01</resolution>
           </range>
@@ -56,5 +56,5 @@
         </ray>
         <plugin name="gazebo_ros_${name}_controller" filename="libgazebo_ros_laser.so">
-          <topicName>scan</topicName>
+          <topicName>/scan</topicName>
           <frameName>${name}_link</frameName>
         </plugin>
