Commit message: Fix

File: vehicle_description/urdf/base.xacro (robot description, xacro)
@@ -1,13 +1,18 @@
 <?xml version="1.0"?>
 <robot xmlns:xacro="http://www.ros.org/wiki/xacro">
-  <xacro:property name="body_length" value="0.95"/>
-  <xacro:property name="body_width" value="0.85"/>
-  <xacro:property name="body_height" value="0.47"/>
+  <!--
+    Scaled‑down chassis for nicer proportions in Gazebo.
+    Original: 0.95 x 0.85 x 0.47 m  |  New: 0.60 x 0.40 x 0.25 m
+  -->
+  <xacro:property name="body_length" value="0.60"/>
+  <xacro:property name="body_width"  value="0.40"/>
+  <xacro:property name="body_height" value="0.25"/>
   <xacro:macro name="base_link">
     <link name="base_link">
       <inertial>
-        <mass value="20.0"/>
+        <mass value="10.0"/>
         <origin xyz="0 0 0"/>
-        <inertia ixx="0.1" ixy="0" ixz="0" iyy="0.1" iyz="0" izz="0.1"/>
+        <!-- simple box inertia approximation -->
+        <inertia ixx="0.05" ixy="0" ixz="0" iyy="0.05" iyz="0" izz="0.05"/>
       </inertial>
       <visual>

File: vehicle_description/urdf/body.xacro (robot description, xacro)
@@ -5,20 +5,21 @@
   <xacro:include filename="$(find vehicle_description)/urdf/differential.xacro"/>
   <xacro:include filename="$(find vehicle_description)/urdf/lidar.xacro"/>
+  <!-- Global constant -->
   <xacro:property name="pi" value="3.1415926535897931" scope="global"/>
   <!-- Base Link -->
   <xacro:base_link/>
-  <!-- Wheels -->
-  <xacro:main_wheel side="left" parent="base_link" xyz="0 0.337 -0.164" rpy="${pi/2} 0 0"/>
-  <xacro:main_wheel side="right" parent="base_link" xyz="0 -0.337 -0.164" rpy="${pi/2} 0 0"/>
-  <!-- Support Wheels -->
-  <xacro:support_wheel name="front_left" parent="base_link" xyz="0.35 0.21 -0.232"/>
-  <xacro:support_wheel name="front_right" parent="base_link" xyz="0.35 -0.21 -0.232"/>
-  <xacro:support_wheel name="rear_left" parent="base_link" xyz="-0.35 0.21 -0.232"/>
-  <xacro:support_wheel name="rear_right" parent="base_link" xyz="-0.35 -0.21 -0.232"/>
-  <!-- Control Systems -->
+  <!-- =====================  Drive Wheels  ===================== -->
+  <!-- Lateral offset ~0.22 m, vertical -0.10 m puts wheel tangent just below chassis -->
+  <xacro:main_wheel side="left"  parent="base_link" xyz="0  0.22 -0.10" rpy="${pi/2} 0 0"/>
+  <xacro:main_wheel side="right" parent="base_link" xyz="0 -0.22 -0.10" rpy="${pi/2} 0 0"/>
+  <!-- =====================  Support Wheels  ===================== -->
+  <!-- front / rear offset 0.25 m, lateral 0.15 m, vertical -0.13 m -->
+  <xacro:support_wheel name="front_left"  parent="base_link" xyz=" 0.25  0.15 -0.13"/>
+  <xacro:support_wheel name="front_right" parent="base_link" xyz=" 0.25 -0.15 -0.13"/>
+  <xacro:support_wheel name="rear_left"   parent="base_link" xyz="-0.25  0.15 -0.13"/>
+  <xacro:support_wheel name="rear_right"  parent="base_link" xyz="-0.25 -0.15 -0.13"/>
+  <!-- =====================  Control & Sensors  ===================== -->
   <xacro:differential_drive/>
-  <!-- IMPORTANT: Add the transmissions -->
   <xacro:wheel_transmissions/>
-  <!-- LiDAR Sensor -->
-  <xacro:lidar_sensor name="hokuyo" parent="base_link" xyz="0.3 0 0.4" rpy="0 0 0"/>
+  <xacro:lidar_sensor name="hokuyo" parent="base_link" xyz="0.23 0 0.30" rpy="0 0 0"/>
 </robot>

File: vehicle_description/urdf/differential.xacro (robot description, xacro)
@@ -2,11 +2,4 @@
 <robot xmlns:xacro="http://www.ros.org/wiki/xacro">
   <xacro:macro name="differential_drive">
-    <!-- Gazebo ROS Control Plugin -->
-    <gazebo>
-      <plugin name="gazebo_ros_control" filename="libgazebo_ros_control.so">
-        <robotNamespace>/</robotNamespace>
-        <robotSimType>gazebo_ros_control/DefaultRobotHWSim</robotSimType>
-      </plugin>
-    </gazebo>
     <!-- Differential Drive Plugin -->
     <gazebo>

File: vehicle_description/urdf/wheels.xacro (robot description, xacro)
@@ -1,15 +1,14 @@
 <?xml version="1.0"?>
 <robot xmlns:xacro="http://www.ros.org/wiki/xacro">
-  <!-- Properties -->
-  <xacro:property name="wheel_radius" value="0.1"/>
-  <xacro:property name="wheel_width" value="0.05"/>
-  <xacro:property name="support_wheel_radius" value="0.029"/>
-  <!-- Main Wheel Macro -->
-  <xacro:macro name="main_wheel" params="side parent xyz rpy">
+  <!-- Scaled wheels -->
+  <xacro:property name="wheel_radius" value="0.08"/>   <!-- was 0.10 -->
+  <xacro:property name="wheel_width"  value="0.04"/>   <!-- was 0.05 -->
+  <xacro:property name="support_wheel_radius" value="0.03"/>
+ <xacro:macro name="main_wheel" params="side parent xyz rpy">
     <link name="${side}_wheel">
       <inertial>
-        <mass value="0.5"/>
+        <mass value="0.3"/>
         <origin xyz="0 0 0"/>
-        <inertia ixx="0.01" ixy="0" ixz="0" iyy="0.01" iyz="0" izz="0.01"/>
+        <inertia ixx="0.005" ixy="0" ixz="0" iyy="0.005" iyz="0" izz="0.005"/>
       </inertial>
       <visual>
@@ -30,18 +29,17 @@
       </gazebo>
     </link>
-    <joint name="${side}_wheel_joint" type="continuous">
-      <parent link="${parent}"/>
-      <child link="${side}_wheel"/>
-      <origin xyz="${xyz}" rpy="${rpy}"/>
-      <axis xyz="0 0 1"/>
+<joint name="${side}_wheel_joint" type="continuous">
+  <parent link="${parent}"/>
+  <child  link="${side}_wheel"/>
+  <origin xyz="${xyz}" rpy="${rpy}"/>
+  <axis xyz="0 1 0"/>
     </joint>
   </xacro:macro>
-  <!-- Support Wheel Macro -->
   <xacro:macro name="support_wheel" params="name parent xyz">
     <link name="${name}_support_wheel">
       <inertial>
-        <mass value="0.1"/>
+        <mass value="0.05"/>
         <origin xyz="0 0 0"/>
-        <inertia ixx="0.001" ixy="0" ixz="0" iyy="0.001" iyz="0" izz="0.001"/>
+        <inertia ixx="0.0005" ixy="0" ixz="0" iyy="0.0005" iyz="0" izz="0.0005"/>
       </inertial>
       <visual>
@@ -66,5 +64,5 @@
       <child link="${name}_support_wheel"/>
       <origin xyz="${xyz}" rpy="0 0 0"/>
-      <axis xyz="1 1 1"/> <!-- Omnidirectional movement -->
+      <axis xyz="1 1 1"/>
     </joint>
   </xacro:macro>
